Commit message: Add gripper.

File: urdf/marvin_pro/marvin_robot.urdf (robot description, URDF)
Before this commit: robot marvin_robot, 30 links, 29 joints
Links:
- link left_gripper_base: geometry collision mesh filename=../../meshes/marvin_pro/meshes/omnigripper/omnigripper_stra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; visual mesh filename=../../meshes/marvin_pro/meshes/omnigripper/omnigripper_stra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
- link left_gripper_left_finger: geometry collision mesh filename=../../meshes/marvin_pro/meshes/omnigripper/Left_Chipper_Bas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; visual mesh filename=../../meshes/marvin_pro/meshes/omnigripper/Left_Chipper_Bas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
- link left_gripper_right_finger: geometry collision mesh filename=../../meshes/marvin_pro/meshes/omnigripper/Right_Chipper_Ba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; visual mesh filename=../../meshes/marvin_pro/meshes/omnigripper/Right_Chipper_Ba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
- link right_gripper_base: geometry collision mesh filename=../../meshes/marvin_pro/meshes/omnigripper/omnigripper_stra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; visual mesh filename=../../meshes/marvin_pro/meshes/omnigripper/omnigripper_stra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
- link right_gripper_left_finger: geometry collision mesh filename=../../meshes/marvin_pro/meshes/omnigripper/Left_Chipper_Bas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; visual mesh filename=../../meshes/marvin_pro/meshes/omnigripper/Left_Chipper_Bas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
- link right_gripper_right_finger: geometry collision mesh filename=../../meshes/marvin_pro/meshes/omnigripper/Right_Chipper_Ba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; visual mesh filename=../../meshes/marvin_pro/meshes/omnigripper/Right_Chipper_Ba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
Joints:
- joint left_gripper_left_finger_joint: origin xyz=0.0516878 -0.0421084 0.0916374 rpy=0.7853982 0 -3.1283863 -> xyz=0.105 -0.0101084 0.0956374 rpy=1.5708 0 3.1416
- joint left_gripper_right_finger_joint: origin xyz=-0.07508 -0.0261034 0.1093149 rpy=2.3561945 0.0000001 0.0132065 -> xyz=-0.05 0.0015034 0.1135 rpy=1.5708 0 0
- joint right_gripper_left_finger_joint: origin xyz=0.0516878 -0.0421084 0.0916374 rpy=0.7853982 0 -3.1283863 -> xyz=0.105 -0.0101084 0.0956374 rpy=1.5708 0 3.1416
- joint right_gripper_right_finger_joint: origin xyz=-0.07508 -0.0261034 0.1093149 rpy=2.3561945 0.0000001 0.0132065 -> xyz=-0.05 0.0015034 0.1135 rpy=1.5708 0 0
