Commit message: Update Robot Description

File: urdf/marvin_pro/marvin_pro_mink_with_45gripper.urdf (robot description, URDF)
Before this commit: robot marvin_robot, 22 links, 21 joints
Links:
- added link left_gripper_base, mass 0.4064271; collision mesh filename=../../meshes/marvin_pro/meshes/45omnigripper/base_link.STL; visual mesh filename=../../meshes/marvin_pro/meshes/45omnigripper/base_link.STL
- added link left_gripper_left_finger, mass 0.031395; collision mesh filename=../../meshes/marvin_pro/meshes/45omnigripper/Left_Finger_Li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; visual mesh filename=../../meshes/marvin_pro/meshes/45omnigripper/Left_Finger_Li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
- added link left_gripper_mount, mass 0
- added link left_gripper_right_finger, mass 0.031395; collision mesh filename=../../meshes/marvin_pro/meshes/45omnigripper/Right_Finger_L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; visual mesh filename=../../meshes/marvin_pro/meshes/45omnigripper/Right_Finger_L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
- added link right_gripper_base, mass 0.4064271; collision mesh filename=../../meshes/marvin_pro/meshes/45omnigripper/base_link.STL; visual mesh filename=../../meshes/marvin_pro/meshes/45omnigripper/base_link.STL
- added link right_gripper_left_finger, mass 0.031395; collision mesh filename=../../meshes/marvin_pro/meshes/45omnigripper/Left_Finger_Li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; visual mesh filename=../../meshes/marvin_pro/meshes/45omnigripper/Left_Finger_Li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
- added link right_gripper_mount, mass 0
- added link right_gripper_right_finger, mass 0.031395; collision mesh filename=../../meshes/marvin_pro/meshes/45omnigripper/Right_Finger_L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; visual mesh filename=../../meshes/marvin_pro/meshes/45omnigripper/Right_Finger_L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
Joints:
- removed joint flange_L_to_left_tool
- removed joint flange_R_to_right_tool
- added joint flange_L_to_left_gripper_mount: type fixed, parent flange_L, child left_gripper_mount, origin xyz=0 0 0 rpy=0 0 -1.5707963
- added joint flange_R_to_right_gripper_mount: type fixed, parent flange_R, child right_gripper_mount, origin xyz=0 0 0 rpy=0 0 -1.5707963
- added joint left_gripper_base_to_left_tool: type fixed, parent left_gripper_base, child left_tool, origin xyz=0 0 0 rpy=0 -1.5707963 -1.5707963
- added joint left_gripper_left_finger_joint: type prismatic, parent left_gripper_base, child left_gripper_left_finger, origin xyz=0.0516878 -0.0421084 0.0916374 rpy=0.7853982 0 -3.1283863, axis 1 0 0, limit lower=0 upper=0.05 effort=30 velocity=0
- added joint left_gripper_mount_to_left_gripper_base: type fixed, parent left_gripper_mount, child left_gripper_base, origin xyz=0 0 0 rpy=0 0 0
- added joint left_gripper_right_finger_joint: type prismatic, parent left_gripper_base, child left_gripper_right_finger, origin xyz=-0.07508 -0.0261034 0.1093149 rpy=2.3561945 0.0000001 0.0132065, axis 1 0 0, limit lower=0 upper=0.05 effort=0 velocity=0, mimic joint=left_gripper_left_finger_joint multiplier=1 offset=0
- added joint right_gripper_base_to_right_tool: type fixed, parent right_gripper_base, child right_tool, origin xyz=0 0 0 rpy=0 -1.5707963 -1.5707963
- added joint right_gripper_left_finger_joint: type prismatic, parent right_gripper_base, child right_gripper_left_finger, origin xyz=0.0516878 -0.0421084 0.0916374 rpy=0.7853982 0 -3.1283863, axis 1 0 0, limit lower=0 upper=0.05 effort=30 velocity=0
- added joint right_gripper_mount_to_right_gripper_base: type fixed, parent right_gripper_mount, child right_gripper_base, origin xyz=0 0 0 rpy=0 0 0
- added joint right_gripper_right_finger_joint: type prismatic, parent right_gripper_base, child right_gripper_right_finger, origin xyz=-0.07508 -0.0261034 0.1093149 rpy=2.3561945 0.0000001 0.0132065, axis 1 0 0, limit lower=0 upper=0.05 effort=0 velocity=0, mimic joint=right_gripper_left_finger_joint multiplier=1 offset=0

File: urdf/marvin_pro/marvin_pro_mink_with_gripper.urdf (robot description, URDF)
Before this commit: robot marvin_robot, 22 links, 21 joints
Links:
- added link left_gripper_base, mass 0.4064271; collision mesh filename=../../meshes/marvin_pro/meshes/omnigripper/omnigripper_stra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; visual mesh filename=../../meshes/marvin_pro/meshes/omnigripper/omnigripper_stra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
- added link left_gripper_left_finger, mass 0.031395; collision mesh filename=../../meshes/marvin_pro/meshes/omnigripper/Left_Chipper_Bas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; visual mesh filename=../../meshes/marvin_pro/meshes/omnigripper/Left_Chipper_Bas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
- added link left_gripper_mount, mass 0
- added link left_gripper_right_finger, mass 0.031395; collision mesh filename=../../meshes/marvin_pro/meshes/omnigripper/Right_Chipper_Ba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; visual mesh filename=../../meshes/marvin_pro/meshes/omnigripper/Right_Chipper_Ba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
- added link right_gripper_base, mass 0.4064271; collision mesh filename=../../meshes/marvin_pro/meshes/omnigripper/omnigripper_stra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; visual mesh filename=../../meshes/marvin_pro/meshes/omnigripper/omnigripper_stra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
- added link right_gripper_left_finger, mass 0.031395; collision mesh filename=../../meshes/marvin_pro/meshes/omnigripper/Left_Chipper_Bas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; visual mesh filename=../../meshes/marvin_pro/meshes/omnigripper/Left_Chipper_Bas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
- added link right_gripper_mount, mass 0
- added link right_gripper_right_finger, mass 0.031395; collision mesh filename=../../meshes/marvin_pro/meshes/omnigripper/Right_Chipper_Ba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; visual mesh filename=../../meshes/marvin_pro/meshes/omnigripper/Right_Chipper_Ba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
Joints:
- removed joint flange_L_to_left_tool
- removed joint flange_R_to_right_tool
- added joint flange_L_to_left_gripper_mount: type fixed, parent flange_L, child left_gripper_mount, origin xyz=0 0 0 rpy=0 0 -1.5707963
- added joint flange_R_to_right_gripper_mount: type fixed, parent flange_R, child right_gripper_mount, origin xyz=0 0 0 rpy=0 0 -1.5707963
- added joint left_gripper_base_to_left_tool: type fixed, parent left_gripper_base, child left_tool, origin xyz=0 0 0 rpy=0 -1.5707963 -1.5707963
- added joint left_gripper_left_finger_joint: type prismatic, parent left_gripper_base, child left_gripper_left_finger, origin xyz=0.105 -0.01 0.0916374 rpy=1.5777046 -0.0094492 -3.1190022, axis 1 0 0, limit lower=0 upper=0.05 effort=30 velocity=0
- added joint left_gripper_mount_to_left_gripper_base: type fixed, parent left_gripper_mount, child left_gripper_base, origin xyz=0 0 0 rpy=0 0 0
- added joint left_gripper_right_finger_joint: type prismatic, parent left_gripper_base, child left_gripper_right_finger, origin xyz=-0.05 -0.002 0.1105 rpy=1.5372318 0.0098779 0.0227581, axis 1 0 0, limit lower=0 upper=0.05 effort=0 velocity=0, mimic joint=left_gripper_left_finger_joint multiplier=1 offset=0
- added joint right_gripper_base_to_right_tool: type fixed, parent right_gripper_base, child right_tool, origin xyz=0 0 0 rpy=0 -1.5707963 -1.5707963
- added joint right_gripper_left_finger_joint: type prismatic, parent right_gripper_base, child right_gripper_left_finger, origin xyz=0.105 -0.01 0.0916374 rpy=1.5777046 -0.0094492 -3.1190022, axis 1 0 0, limit lower=0 upper=0.05 effort=30 velocity=0
- added joint right_gripper_mount_to_right_gripper_base: type fixed, parent right_gripper_mount, child right_gripper_base, origin xyz=0 0 0 rpy=0 0 0
- added joint right_gripper_right_finger_joint: type prismatic, parent right_gripper_base, child right_gripper_right_finger, origin xyz=-0.05 -0.002 0.1105 rpy=1.5372318 0.0098779 0.0227581, axis 1 0 0, limit lower=0 upper=0.05 effort=0 velocity=0, mimic joint=right_gripper_left_finger_joint multiplier=1 offset=0
